Commit message: Added TM12 model and included transform points into rviz for view_pick and view_place

File: install/tmr_description/share/tmr_description/xacro/gripper/robotiq_2f.urdf.xacro (robot description, xacro)
@@ -1,59 +1 @@
-<?xml version="1.0"?>
-<robot xmlns:xacro="http://www.ros.org/wiki/xacro" name="gripper" >
-  <xacro:include filename="$(find tmr_description)/xacro/gripper/robotiq_85_gripper.urdf.xacro"/>
-  <xacro:macro name="robotiq_2f" params="prefix">
-    <!--  + Reference frame: at the middle (4mm) -->
-  <link name="robotiq_coupler">
-    <visual>
-      <geometry>
-        <mesh filename="package://tmr_description/meshes/gripper/robotiq/2f-85/robotiq_85_coupler.stl" />
-      </geometry>
-      <material name="white"/>
-    </visual>
-    <collision>
-      <geometry>
-        <mesh filename="package://tmr_description/meshes/gripper/robotiq/2f-85/robotiq_85_coupler.stl" />
-      </geometry>
-    </collision>
-    <inertial>
-      <origin xyz="2.073e-05   1.45286e-03  -1.1049e-03" rpy="0 0 0" />
-      <mass value="0.168" />
-      <inertia ixx="6.69695624e-05" ixy="5.21511788e-09" ixz="-2.74383009e-08"
-               iyy="7.85088161e-05" iyz="5.41105193e-07" izz="1.41819717e-04"/>
-    </inertial>
-  </link>
-  <joint name="robotiq_coupler_joint" type="fixed">
-    <origin xyz="0 0 0.004" rpy="0 0 ${-pi/2.0}" />
-    <parent link="${prefix}flange"/>
-    <child link="robotiq_coupler"/>
-  </joint>
-  <gazebo reference="robotiq_coupler">
-    <mu1>0.9</mu1>
-    <mu2>0.9</mu2>
-    <material>Gazebo/FlatBlack</material>
-  </gazebo>
-  <!-- Equivalent to the OpenRAVE manipulator denso_robotiq_85_gripper -->
-  <!-- <link name="denso_robotiq_85_gripper" /> -->
-  <!-- <joint name="manipulator_dummy_joint" type="fixed"> -->
-  <!--   <origin xyz="0 0 0.1441" rpy="0 0 0" /> -->
-  <!--   <parent link="robotiq_coupler"/> -->
-  <!--   <child link="denso_robotiq_85_gripper"/> -->
-  <!-- </joint> -->
-  <!-- Attach the robotiq 85 gripper -->
-  <xacro:robotiq_85_gripper prefix="" parent="robotiq_coupler" >
-    <origin xyz="0 0 0.004" rpy="0 ${-pi/2} ${pi}"/>
-  </xacro:robotiq_85_gripper>
-  <gazebo>
-    <gripper name="gazebo_gripper">
-      <grasp_check>
-        <attach_steps>2</attach_steps>    <!-- default: 20 -->
-        <detach_steps>2</detach_steps>    <!-- default: 40 -->
-        <min_contact_count>3</min_contact_count>
-      </grasp_check>
-      <gripper_link>robotiq_85_left_finger_tip_link</gripper_link>
-      <gripper_link>robotiq_85_right_finger_tip_link</gripper_link>
-      <palm_link>robotiq_85_base_link</palm_link>
-    </gripper>
-  </gazebo>
-  </xacro:macro>
-</robot>
+/home/gy/Omron_TM_ROS2/tmr_description/xacro/gripper/robotiq_2f.urdf.xacro

File: install/tmr_description/share/tmr_description/xacro/gripper/robotiq_85_gripper.transmission.xacro (robot description, xacro)
@@ -1,44 +1 @@
-<?xml version="1.0"?>
-<robot xmlns:xacro="http://www.ros.org/wiki/xacro">
-  <xacro:macro name="robotiq_85_gripper_transmission" params="prefix">
-    <transmission name="${prefix}robotiq_85_left_knuckle_trans">
-      <type>transmission_interface/SimpleTransmission</type>
-      <joint name="${prefix}robotiq_85_left_knuckle_joint">
-        <hardwareInterface>hardware_interface/PositionJointInterface</hardwareInterface>
-        <!-- <hardwareInterface>EffortJointInterface</hardwareInterface> -->
-      </joint>
-      <actuator name="${prefix}robotiq_85_left_knuckle_motor">
-        <mechanicalReduction>1</mechanicalReduction>
-        <hardwareInterface>hardware_interface/PositionJointInterface</hardwareInterface>
-        <!-- <hardwareInterface>EfforJointInterface</hardwareInterface> -->
-      </actuator>
-    </transmission>
-    <!-- Mimic joints -->
-    <gazebo>
-      <plugin filename="libgazebo_mimic_joint_plugin.so" name="${prefix}mimic_robotiq_85_1">
-        <joint>${prefix}robotiq_85_left_knuckle_joint</joint>
-        <mimicJoint>${prefix}robotiq_85_right_knuckle_joint</mimicJoint>
-      </plugin>
-      <plugin filename="libgazebo_mimic_joint_plugin.so" name="${prefix}mimic_robotiq_85_2">
-        <joint>${prefix}robotiq_85_left_knuckle_joint</joint>
-        <mimicJoint>${prefix}robotiq_85_left_inner_knuckle_joint</mimicJoint>
-      </plugin>
-      <plugin filename="libgazebo_mimic_joint_plugin.so" name="${prefix}mimic_robotiq_85_3">
-        <joint>${prefix}robotiq_85_left_knuckle_joint</joint>
-        <mimicJoint>${prefix}robotiq_85_right_inner_knuckle_joint</mimicJoint>
-      </plugin>
-      <plugin filename="libgazebo_mimic_joint_plugin.so" name="${prefix}mimic_robotiq_85_4">
-        <joint>${prefix}robotiq_85_left_knuckle_joint</joint>
-        <mimicJoint>${prefix}robotiq_85_left_finger_tip_joint</mimicJoint>
-        <multiplier>-1.0</multiplier>
-        <offset>0.0</offset>
-      </plugin>
-      <plugin filename="libgazebo_mimic_joint_plugin.so" name="${prefix}mimic_robotiq_85_5">
-        <joint>${prefix}robotiq_85_left_knuckle_joint</joint>
-        <mimicJoint>${prefix}robotiq_85_right_finger_tip_joint</mimicJoint>
-        <multiplier>-1.0</multiplier>
-        <offset>0.0</offset>
-      </plugin>
-    </gazebo>
-  </xacro:macro>
-</robot>
+/home/gy/Omron_TM_ROS2/tmr_description/xacro/gripper/robotiq_85_gripper.transmission.xacro

File: install/tmr_description/share/tmr_description/xacro/gripper/robotiq_85_gripper.urdf.xacro (robot description, xacro)
@@ -1,257 +1 @@
-<?xml version="1.0"?>
-<robot name="robotiq_85_gripper" xmlns:xacro="http://www.ros.org/wiki/xacro">
-  <xacro:include filename="$(find tmr_description)/xacro/gripper/robotiq_85_gripper.transmission.xacro" />
-  <xacro:macro name="robotiq_85_gripper" params="prefix parent *origin">
-    <joint name="${prefix}robotiq_85_base_joint" type="fixed">
-      <parent link="${parent}"/>
-      <child link="${prefix}robotiq_85_base_link"/>
-      <xacro:insert_block name="origin"/>
-    </joint>
-    <link name="${prefix}robotiq_85_base_link">
-      <visual>
-        <geometry>
-          <mesh filename="package://tmr_description/meshes/gripper/robotiq/2f-85/visual/robotiq_85_base_link.dae"/>
-        </geometry>
-      </visual>
-      <collision>
-        <geometry>
-          <mesh filename="package://tmr_description/meshes/gripper/robotiq/2f-85/collision/robotiq_85_base_link.stl"/>
-        </geometry>
-      </collision>
-      <inertial>
-        <mass value="0.636951" />
-        <origin xyz="0.0 0.0 0.0" />
-        <inertia ixx = "0.000380" ixy = "0.000000" ixz = "0.000000"
-             iyx = "0.000000" iyy = "0.001110" iyz = "0.000000"
-             izx = "0.000000" izy = "0.000000" izz = "0.001171" />
-      </inertial>
-    </link>
-    <joint name="${prefix}robotiq_85_left_knuckle_joint" type="revolute">
-      <parent link="${prefix}robotiq_85_base_link"/>
-      <child link="${prefix}robotiq_85_left_knuckle_link"/>
-      <axis xyz="0 0 1"/>
-      <origin rpy="${pi} 0.0 0.0" xyz="0.05490451627 0.03060114443 0.0"/>
-      <limit lower="0.0" upper="0.80285" velocity="0.5" effort="1000"/>
-    </joint>
-    <joint name="${prefix}robotiq_85_right_knuckle_joint" type="continuous">
-      <parent link="${prefix}robotiq_85_base_link"/>
-      <child link="${prefix}robotiq_85_right_knuckle_link"/>
-      <axis xyz="0 0 1"/>
-      <origin rpy="0.0 0.0 0.0" xyz="0.05490451627 -0.03060114443 0.0"/>
-      <limit lower="-3.14" upper="3.14" velocity="100.0" effort="1000"/>
-      <mimic joint="${prefix}robotiq_85_left_knuckle_joint"/>
-    </joint>
-    <link name="${prefix}robotiq_85_left_knuckle_link">
-      <visual>
-        <geometry>
-          <mesh filename="package://tmr_description/meshes/gripper/robotiq/2f-85/visual/robotiq_85_knuckle_link.dae"/>
-        </geometry>
-      </visual>
-      <collision>
-        <geometry>
-          <mesh filename="package://tmr_description/meshes/gripper/robotiq/2f-85/collision/robotiq_85_knuckle_link.stl"/>
-        </geometry>
-      </collision>
-      <inertial>
-        <mass value="0.018491" />
-        <origin xyz="0.0 0.0 0.0" />
-        <inertia ixx = "0.000009" ixy = "-0.000001" ixz = "0.000000"
-             iyx = "-0.000001" iyy = "0.000001" iyz = "0.000000"
-             izx = "0.000000" izy = "0.000000" izz = "0.000010" />
-      </inertial>
-    </link>
-    <link name="${prefix}robotiq_85_right_knuckle_link">
-      <visual>
-        <geometry>
-          <mesh filename="package://tmr_description/meshes/gripper/robotiq/2f-85/visual/robotiq_85_knuckle_link.dae"/>
-        </geometry>
-      </visual>
-      <collision>
-        <geometry>
-          <mesh filename="package://tmr_description/meshes/gripper/robotiq/2f-85/collision/robotiq_85_knuckle_link.stl"/>
-        </geometry>
-      </collision>
-      <inertial>
-        <mass value="0.018491" />
-        <origin xyz="0.0 0.0 0.0" />
-        <inertia ixx = "0.000009" ixy = "-0.000001" ixz = "0.000000"
-             iyx = "-0.000001" iyy = "0.000001" iyz = "0.000000"
-             izx = "0.000000" izy = "0.000000" izz = "0.000010" />
-      </inertial>
-    </link>
-    <joint name="${prefix}robotiq_85_left_finger_joint" type="fixed">
-      <parent link="${prefix}robotiq_85_left_knuckle_link"/>
-      <child link="${prefix}robotiq_85_left_finger_link"/>
-      <origin xyz="-0.00408552455 -0.03148604435 0.0" rpy="0 0 0" />
-    </joint>
-    <joint name="${prefix}robotiq_85_right_finger_joint" type="fixed">
-      <parent link="${prefix}robotiq_85_right_knuckle_link"/>
-      <child link="${prefix}robotiq_85_right_finger_link"/>
-      <origin xyz="-0.00408552455 -0.03148604435 0.0" rpy="0 0 0" />
-    </joint>
-    <link name="${prefix}robotiq_85_left_finger_link">
-      <visual>
-        <geometry>
-          <mesh filename="package://tmr_description/meshes/gripper/robotiq/2f-85/visual/robotiq_85_finger_link.dae"/>
-        </geometry>
-      </visual>
-      <collision>
-        <geometry>
-          <mesh filename="package://tmr_description/meshes/gripper/robotiq/2f-85/collision/robotiq_85_finger_link.stl"/>
-        </geometry>
-      </collision>
-      <inertial>
-        <mass value="0.027309" />
-        <origin xyz="0.0 0.0 0.0" />
-        <inertia ixx = "0.000003" ixy = "-0.000002" ixz = "0.000000"
-             iyx = "-0.000002" iyy = "0.000021" iyz = "0.000000"
-             izx = "0.000000" izy = "0.000000" izz = "0.000020" />
-      </inertial>
-    </link>
-    <link name="${prefix}robotiq_85_right_finger_link">
-      <visual>
-        <geometry>
-          <mesh filename="package://tmr_description/meshes/gripper/robotiq/2f-85/visual/robotiq_85_finger_link.dae"/>
-        </geometry>
-      </visual>
-      <collision>
-        <geometry>
-          <mesh filename="package://tmr_description/meshes/gripper/robotiq/2f-85/collision/robotiq_85_finger_link.stl"/>
-        </geometry>
-      </collision>
-      <inertial>
-        <mass value="0.027309" />
-        <origin xyz="0.0 0.0 0.0" />
-        <inertia ixx = "0.000003" ixy = "-0.000002" ixz = "0.000000"
-             iyx = "-0.000002" iyy = "0.000021" iyz = "0.000000"
-             izx = "0.000000" izy = "0.000000" izz = "0.000020" />
-      </inertial>
-    </link>
-    <joint name="${prefix}robotiq_85_left_inner_knuckle_joint" type="continuous">
-      <parent link="${prefix}robotiq_85_base_link"/>
-      <child link="${prefix}robotiq_85_left_inner_knuckle_link"/>
-      <axis xyz="0 0 1"/>
-      <origin xyz="0.06142 0.0127 0" rpy="${pi} 0.0 0.0" />
-      <limit lower="-3.14" upper="3.14" velocity="100.0" effort="0.1"/>
-      <mimic joint="${prefix}robotiq_85_left_knuckle_joint" offset="0"/>
-    </joint>
-    <joint name="${prefix}robotiq_85_right_inner_knuckle_joint" type="continuous">
-      <parent link="${prefix}robotiq_85_base_link"/>
-      <child link="${prefix}robotiq_85_right_inner_knuckle_link"/>
-      <axis xyz="0 0 1"/>
-      <origin xyz="0.06142 -0.0127 0" rpy="0 0 0"/>
-      <limit lower="-3.14" upper="3.14" velocity="100.0" effort="0.1"/>
-      <mimic joint="${prefix}robotiq_85_left_knuckle_joint" offset="0"/>
-    </joint>
-    <link name="${prefix}robotiq_85_left_inner_knuckle_link">
-      <visual>
-        <geometry>
-          <mesh filename="package://tmr_description/meshes/gripper/robotiq/2f-85/visual/robotiq_85_inner_knuckle_link.dae"/>
-        </geometry>
-      </visual>
-      <collision>
-        <geometry>
-          <mesh filename="package://tmr_description/meshes/gripper/robotiq/2f-85/collision/robotiq_85_inner_knuckle_link.stl"/>
-        </geometry>
-      </collision>
-      <inertial>
-        <mass value="0.029951" />
-        <origin xyz="0.0 0.0 0.0" />
-        <inertia ixx = "0.000039" ixy = "0.000000" ixz = "0.000000"
-             iyx = "0.000000" iyy = "0.000005" iyz = "0.000000"
-             izx = "0.000000" izy = "0.000000" izz = "0.000035" />
-      </inertial>
-    </link>
-    <link name="${prefix}robotiq_85_right_inner_knuckle_link">
-      <visual>
-        <geometry>
-          <mesh filename="package://tmr_description/meshes/gripper/robotiq/2f-85/visual/robotiq_85_inner_knuckle_link.dae"/>
-        </geometry>
-      </visual>
-      <collision>
-        <geometry>
-          <mesh filename="package://tmr_description/meshes/gripper/robotiq/2f-85/collision/robotiq_85_inner_knuckle_link.stl"/>
-        </geometry>
-      </collision>
-      <inertial>
-        <mass value="0.029951" />
-        <origin xyz="0.0 0.0 0.0" />
-        <inertia ixx = "0.000039" ixy = "0.000000" ixz = "0.000000"
-             iyx = "0.000000" iyy = "0.000005" iyz = "0.000000"
-             izx = "0.000000" izy = "0.000000" izz = "0.000035" />
-      </inertial>
-    </link>
-    <joint name="${prefix}robotiq_85_left_finger_tip_joint" type="continuous">
-      <parent link="${prefix}robotiq_85_left_inner_knuckle_link"/>
-      <child link="${prefix}robotiq_85_left_finger_tip_link"/>
-      <axis xyz="0 0 1"/>
-      <origin xyz="0.04303959807 -0.03759940821 0.0" rpy="0.0 0.0 0.0"/>
-      <limit lower="-3.14" upper="3.14" velocity="100.0" effort="0.1"/>
-      <mimic joint="${prefix}robotiq_85_left_knuckle_joint" multiplier="-1"/>
-    </joint>
-    <joint name="${prefix}robotiq_85_right_finger_tip_joint" type="continuous">
-      <parent link="${prefix}robotiq_85_right_inner_knuckle_link"/>
-      <child link="${prefix}robotiq_85_right_finger_tip_link"/>
-      <axis xyz="0 0 1"/>
-      <origin rpy="0.0 0.0 0.0" xyz="0.04303959807 -0.03759940821  0.0"/>
-      <limit lower="-3.14" upper="3.14" velocity="100.0" effort="0.1"/>
-      <mimic joint="${prefix}robotiq_85_left_knuckle_joint" multiplier="-1"/>
-    </joint>
-    <link name="${prefix}robotiq_85_left_finger_tip_link">
-      <visual>
-        <geometry>
-          <mesh filename="package://tmr_description/meshes/gripper/robotiq/2f-85/visual/robotiq_85_finger_tip_link.dae"/>
-        </geometry>
-      </visual>
-      <dynamics damping="0.0" friction="100.0"/>
-      <collision>
-        <geometry>
-          <mesh filename="package://tmr_description/meshes/gripper/robotiq/2f-85/collision/robotiq_85_finger_tip_link.stl"/>
-        </geometry>
-      </collision>
-      <inertial>
-        <mass value="0.019555" />
-        <origin xyz="0.0 0.0 0.0" />
-        <inertia ixx = "0.000002" ixy = "0.000000" ixz = "0.000000"
-             iyx = "0.000000" iyy = "0.000005" iyz = "0.000000"
-             izx = "0.000000" izy = "0.000000" izz = "0.000006" />
-      </inertial>
-    </link>
-    <link name="${prefix}robotiq_85_right_finger_tip_link">
-      <visual>
-        <geometry>
-          <mesh filename="package://tmr_description/meshes/gripper/robotiq/2f-85/visual/robotiq_85_finger_tip_link.dae"/>
-        </geometry>
-      </visual>
-      <dynamics damping="0.0" friction="100.0"/>
-      <collision>
-        <geometry>
-          <mesh filename="package://tmr_description/meshes/gripper/robotiq/2f-85/collision/robotiq_85_finger_tip_link.stl"/>
-        </geometry>
-      </collision>
-      <inertial>
-        <mass value="0.019555" />
-        <origin xyz="0.0 0.0 0.0" />
-        <inertia ixx = "0.000002" ixy = "0.000000" ixz = "0.000000"
-             iyx = "0.000000" iyy = "0.000005" iyz = "0.000000"
-             izx = "0.000000" izy = "0.000000" izz = "0.000006" />
-      </inertial>
-    </link>
-    <!-- Improve grasping physics -->
-    <gazebo reference="${prefix}robotiq_85_left_finger_tip_link">
-      <kp>1000000.0</kp>
-      <kd>1.0</kd>
-      <mu1>100</mu1>
-      <mu2>100</mu2>
-      <minDepth>0.001</minDepth>
-    </gazebo>
-    <gazebo reference="${prefix}robotiq_85_right_finger_tip_link">
-      <kp>1000000.0</kp>
-      <kd>1.0</kd>
-      <mu1>100</mu1>
-      <mu2>100</mu2>
-      <minDepth>0.001</minDepth>
-    </gazebo>
-    <xacro:robotiq_85_gripper_transmission prefix="${prefix}" />
-  </xacro:macro>
-</robot>
+/home/gy/Omron_TM_ROS2/tmr_description/xacro/gripper/robotiq_85_gripper.urdf.xacro

File: install/tmr_description/share/tmr_description/xacro/gripper/robotiq_85_gripper.xacro (robot description, xacro)
@@ -1,39 +1 @@
-<?xml version="1.0" ?>
-<robot name="robotiq_85_gripper" xmlns:xacro="http://www.ros.org/wiki/xacro">
-  <xacro:include filename="$(find dsr_description)/xacro/robotiq_85_gripper.urdf.xacro" />
-  <gazebo>
-    <plugin name="gazebo_ros_control" filename="libgazebo_ros_control.so">
-      <robotNamespace>/</robotNamespace>
-    </plugin>
-  </gazebo>
-  <link name="world"/>
-  <joint name="world_fixed" type="fixed">
-    <origin xyz="0 0 0" rpy="0 0 0"/>
-    <parent link="world"/>
-    <child link="gripper_root_link"/>
-  </joint>
-  <link name="gripper_root_link">
-    <visual>
-      <origin xyz="0 0 0.5" rpy="0 0 0"/>
-      <geometry>
-        <box size="0.1 0.1 1.0"/>
-      </geometry>
-    </visual>
-    <collision>
-      <origin xyz="0 0 0.5" rpy="0 0 0"/>
-      <geometry>
-        <box size="0.1 0.1 1.0"/>
-      </geometry>
-    </collision>
-    <inertial>
-      <mass value="1e2" />
-      <origin xyz="0.0 0.0 0.0" />
-      <inertia ixx = "0.000001" ixy = "0.000000" ixz = "0.000000"
-           iyx = "0.000000" iyy = "0.000001" iyz = "0.000000"
-           izx = "0.000000" izy = "0.000000" izz = "0.000001" />
-    </inertial>
-  </link>
-  <xacro:robotiq_85_gripper prefix="" parent="gripper_root_link" >
-    <origin xyz="0.05 0 0.85" rpy="0 0 0"/>
-  </xacro:robotiq_85_gripper>
-</robot>
+/home/gy/Omron_TM_ROS2/tmr_description/xacro/gripper/robotiq_85_gripper.xacro

File: install/tmr_description/share/tmr_description/xacro/gripper/robotiq_85_gripper_sim_base.urdf.xacro (robot description, xacro)
@@ -1,26 +1 @@
-<?xml version="1.0"?>
-<robot name="robotiq_85_gripper_sim_base" xmlns:xacro="http://www.ros.org/wiki/xacro">
-  <xacro:macro name="robotiq_85_gripper_sim_base" params="prefix">
-    <link name="${prefix}gripper_root_link">
-      <visual>
-        <origin xyz="0.05 0.05 0.5" rpy="0 0 0"/>
-        <geometry>
-          <box size="0.1 0.1 1.0"/>
-        </geometry>
-      </visual>
-      <collision>
-        <origin xyz="0.05 0.05 0.5" rpy="0 0 0"/>
-        <geometry>
-          <box size="0.1 0.1 1.0"/>
-        </geometry>
-      </collision>
-      <inertial>
-        <mass value="1e2" />
-        <origin xyz="0.0 0.0 0.0" />
-        <inertia ixx = "0.000001" ixy = "0.000000" ixz = "0.000000"
-             iyx = "0.000000" iyy = "0.000001" iyz = "0.000000"
-             izx = "0.000000" izy = "0.000000" izz = "0.000001" />
-      </inertial>
-    </link>
-  </xacro:macro>
-</robot>
+/home/gy/Omron_TM_ROS2/tmr_description/xacro/gripper/robotiq_85_gripper_sim_base.urdf.xacro

File: install/tmr_description/share/tmr_description/xacro/macro.gazebo.xacro (robot description, xacro)
@@ -1,29 +1 @@
-<?xml version="1.0"?>
-<robot xmlns:xacro="http://wiki.ros.org/xacro">
-  <xacro:macro name="tmr_gazebo" params="ns prefix">
-    <gazebo reference="${prefix}link_1">
-      <selfCollide>true</selfCollide>
-    </gazebo>
-    <gazebo reference="${prefix}link_2">
-      <selfCollide>true</selfCollide>
-    </gazebo>
-    <gazebo reference="${prefix}link_3">
-      <selfCollide>true</selfCollide>
-    </gazebo>
-    <gazebo reference="${prefix}link_4">
-      <selfCollide>true</selfCollide>
-    </gazebo>
-    <gazebo reference="${prefix}link_5">
-      <selfCollide>true</selfCollide>
-    </gazebo>
-    <gazebo reference="${prefix}link_6">
-      <selfCollide>true</selfCollide>
-    </gazebo>
-    <gazebo>
-      <plugin name="gazebo_ros_control" filename="libgazebo_ros_control.so">
-        <robotNamespace>/${ns}</robotNamespace>
-        <robotSimType>gazebo_ros_control/DefaultRobotHWSim</robotSimType>
-      </plugin>
-    </gazebo>
-  </xacro:macro>
-</robot>
+/home/gy/Omron_TM_ROS2/tmr_description/xacro/macro.gazebo.xacro

File: install/tmr_description/share/tmr_description/xacro/macro.inertial.xacro (robot description, xacro)
@@ -1,33 +1 @@
-<?xml version="1.0"?>
-<robot xmlns:xacro="http://wiki.ros.org/xacro">
-  <xacro:macro name="cylinder_inertial_x" params="radius length mass *origin">
-    <inertial>
-      <mass value="${mass}" />
-      <xacro:insert_block name="origin" />
-      <inertia
-        ixx="${0.5 * mass * radius * radius}" ixy="0.0" ixz="0.0"
-        iyy="${0.0833333 * mass * (3 * radius * radius + length * length)}" iyz="0.0"
-        izz="${0.0833333 * mass * (3 * radius * radius + length * length)}" />
-    </inertial>
-  </xacro:macro>
-  <xacro:macro name="cylinder_inertial_y" params="radius length mass *origin">
-    <inertial>
-      <mass value="${mass}" />
-      <xacro:insert_block name="origin" />
-      <inertia
-        ixx="${0.0833333 * mass * (3 * radius * radius + length * length)}" ixy="0.0" ixz="0.0"
-        iyy="${0.5 * mass * radius * radius}" iyz="0.0"
-        izz="${0.0833333 * mass * (3 * radius * radius + length * length)}" />
-    </inertial>
-  </xacro:macro>
-  <xacro:macro name="cylinder_inertial_z" params="radius length mass *origin">
-    <inertial>
-      <mass value="${mass}" />
-      <xacro:insert_block name="origin" />
-      <inertia
-        ixx="${0.0833333 * mass * (3 * radius * radius + length * length)}" ixy="0.0" ixz="0.0"
-        iyy="${0.0833333 * mass * (3 * radius * radius + length * length)}" iyz="0.0"
-        izz="${0.5 * mass * radius * radius}" />
-    </inertial>
-  </xacro:macro>
-</robot>
+/home/gy/Omron_TM_ROS2/tmr_description/xacro/macro.inertial.xacro
