Commit message: Added TM12 model and included transform points into rviz for view_pick and view_place

File: install/tmr_description/share/tmr_description/xacro/macro.materials.xacro (robot description, xacro)
@@ -1,35 +1 @@
-<?xml version="1.0"?>
-<robot xmlns:xacro="http://www.ros.org/wiki/xacro">
-	<xacro:macro name="tmr_materials">
-    <material name="grey">
-			<color rgba="0.5 0.5 0.5 1.0" />
-		</material>
-		<material name="white">
-			<color rgba="0.95 0.95 0.95 1.0" />
-		</material>
-		<material name="red">
-			<color rgba="0.95 0.0 0.0 1.0" />
-		</material>
-		<material name="orange">
-			<color rgba="1.0 0.5 0.0 1.0" />
-		</material>
-		<material name="yellow">
-			<color rgba="1.0 1.0 0.0 1.0" />
-		</material>
-		<material name="green">
-			<color rgba="0.0 1.0 0.0 1.0" />
-		</material>
-		<material name="blue">
-			<color rgba="0.0 0.0 1.0 1.0" />
-		</material>
-		<material name="indigo">
-			<color rgba="0.3 0.3 0.6 1.0" />
-		</material>
-		<material name="violet">
-			<color rgba="0.6 0.0 1.0 1.0" />
-		</material>
-		<material name="black">
-			<color rgba="0.0 0.0 0.0 1.0" />
-		</material>
-	</xacro:macro>
-</robot>
+/home/gy/Omron_TM_ROS2/tmr_description/xacro/macro.materials.xacro

File: install/tmr_description/share/tmr_description/xacro/macro.tm5-900.urdf.xacro (robot description, xacro)
@@ -1,200 +1 @@
-<?xml version="1.0"?>
-<robot xmlns:xacro="http://wiki.ros.org/xacro">
-  <xacro:include filename="$(find tmr_description)/xacro/macro.inertial.xacro" />
-  <xacro:macro name="tm5-900" params="ns prefix
-    color:=none format:=obj">
-<!--
-    <xacro:property name="shoulder_offset" value="0.146" />
-    <xacro:property name="elbow_offset" value="0.1297" />
-    <xacro:property name="wrist_offset" value="0.106" />
--->
-    <xacro:property name="mass_0" value="1.0" />
-    <xacro:property name="mass_1" value="4.5" />
-    <xacro:property name="mass_2" value="11.0" />
-    <xacro:property name="mass_3" value="2.5" />
-    <xacro:property name="mass_4" value="1.45" />
-    <xacro:property name="mass_5" value="1.45" />
-    <xacro:property name="mass_6" value="0.4" />
-<!--LinkDescription-->
-  <link name="${prefix}link_0">
-    <visual>
-      <geometry>
-        <mesh filename="package://tmr_description/meshes/tm5-900/visual/tm5_base.${format}" />
-      </geometry>
-      <material name="${color}" />
-    </visual>
-    <collision>
-      <geometry>
-        <mesh filename="package://tmr_description/meshes/tm5-900/collision/tm5_base_c.stl" />
-      </geometry>
-    </collision>
-<!--inertial-->
-    <xacro:cylinder_inertial_z radius="0.06" length="0.05" mass="${mass_0}">
-      <origin xyz="0 0 0" rpy="0 0 0" />
-    </xacro:cylinder_inertial_z>
-  </link>
-  <joint name="${prefix}joint_1" type="revolute">
-    <parent link="${prefix}link_0" />
-    <child link="${prefix}link_1" />
-    <origin xyz="0 0 0.1452" rpy="0 0 0" />
-    <axis xyz="0 0 1" />
-<!--limit-->
-    <limit lower="${-1.5*pi}" upper="${1.5*pi}" velocity="3.14" effort="320.0" />
-  </joint>
-  <link name="${prefix}link_1">
-    <visual>
-      <geometry>
-        <mesh filename="package://tmr_description/meshes/tm5-900/visual/tmr_400w_01.${format}" />
-      </geometry>
-      <material name="${color}" />
-    </visual>
-    <collision>
-      <geometry>
-        <mesh filename="package://tmr_description/meshes/tm5-900/collision/tmr_400w_01_c.stl" />
-      </geometry>
-    </collision>
-<!--inertial-->
-    <xacro:cylinder_inertial_z radius="0.06" length="0.15" mass="${mass_1}">
-      <origin xyz="0 0 0" rpy="0 0 0" />
-    </xacro:cylinder_inertial_z>
-  </link>
-  <joint name="${prefix}joint_2" type="revolute">
-    <parent link="${prefix}link_1" />
-    <child link="${prefix}link_2" />
-    <origin xyz="0 0 0" rpy="${-0.5*pi} ${-0.5*pi} 0" />
-    <axis xyz="0 0 1" />
-<!--limit-->
-    <limit lower="${-pi}" upper="${pi}" velocity="3.14" effort="320" />
-  </joint>
-  <link name="${prefix}link_2">
-    <visual>
-      <geometry>
-        <mesh filename="package://tmr_description/meshes/tm5-900/visual/tm5-900_arm1.${format}" />
-      </geometry>
-      <material name="${color}" />
-    </visual>
-    <collision>
-      <geometry>
-        <mesh filename="package://tmr_description/meshes/tm5-900/collision/tm5-900_arm1_c.stl" />
-      </geometry>
-    </collision>
-<!--inertial-->
-    <xacro:cylinder_inertial_x radius="0.06" length="0.429" mass="${mass_2}">
-      <origin xyz="0.2145 0 -0.146" rpy="0 0 0" />
-    </xacro:cylinder_inertial_x>
-  </link>
-  <joint name="${prefix}joint_3" type="revolute">
-    <parent link="${prefix}link_2" />
-    <child link="${prefix}link_3" />
-    <origin  xyz="0.429 0 0" rpy="0 0 0" />
-    <axis xyz="0 0 1" />
-<!--limit-->
-    <limit lower="${-pi}" upper="${pi}" velocity="3.14" effort="320" />
-  </joint>
-  <link name="${prefix}link_3">
-    <visual>
-      <geometry>
-        <mesh filename="package://tmr_description/meshes/tm5-900/visual/tm5-900_arm2.${format}" />
-      </geometry>
-      <material name="${color}" />
-    </visual>
-    <collision>
-      <geometry>
-        <mesh filename="package://tmr_description/meshes/tm5-900/collision/tm5-900_arm2_c.stl" />
-      </geometry>
-    </collision>
-<!--inertial-->
-    <xacro:cylinder_inertial_x radius="0.045" length="0.4115" mass="${mass_3}">
-      <origin xyz="0.20575 0 -0.0163" rpy="0 0 0" />
-    </xacro:cylinder_inertial_x>
-  </link>
-  <joint name="${prefix}joint_4" type="revolute">
-    <parent link="${prefix}link_3" />
-    <child link="${prefix}link_4" />
-    <origin xyz="0.4115 0 -0.1223" rpy="0 0 ${0.5*pi}" />
-    <axis xyz="0 0 1" />
-<!--limit-->
-    <limit lower="${-pi}" upper="${pi}" velocity="3.92" effort="80" />
-  </joint>
-  <link name="${prefix}link_4">
-    <visual>
-      <geometry>
-        <mesh filename="package://tmr_description/meshes/tm5-900/visual/tmr_100w_01.${format}" />
-      </geometry>
-      <material name="${color}" />
-    </visual>
-    <collision>
-      <geometry>
-        <mesh filename="package://tmr_description/meshes/tm5-900/collision/tmr_100w_01_c.stl" />
-      </geometry>
-    </collision>
-<!--inertial-->
-    <xacro:cylinder_inertial_y radius="0.045" length="0.12" mass="${mass_4}">
-      <origin xyz="0 0 0" rpy="0 0 0" />
-    </xacro:cylinder_inertial_y>
-  </link>
-  <joint name="${prefix}joint_5" type="revolute">
-    <parent link="${prefix}link_4" />
-    <child link="${prefix}link_5" />
-    <origin xyz="0 -0.106 0" rpy="${0.5*pi} 0 0" />
-    <axis xyz="0 0 1" />
-<!--limit-->
-    <limit lower="${-pi}" upper="${pi}" velocity="3.92" effort="80" />
-  </joint>
-  <link name="${prefix}link_5">
-    <visual>
-      <geometry>
-        <mesh filename="package://tmr_description/meshes/tm5-900/visual/tmr_100w_02.${format}" />
-      </geometry>
-      <material name="${color}" />
-    </visual>
-    <collision>
-      <geometry>
-        <mesh filename="package://tmr_description/meshes/tm5-900/collision/tmr_100w_02_c.stl" />
-      </geometry>
-    </collision>
-<!--inertial-->
-    <xacro:cylinder_inertial_y radius="0.045" length="0.12" mass="${mass_5}">
-      <origin xyz="0 0 0" rpy="0 0 0" />
-    </xacro:cylinder_inertial_y>
-  </link>
-  <joint name="${prefix}joint_6" type="revolute">
-    <parent link="${prefix}link_5" />
-    <child link="${prefix}link_6" />
-    <origin xyz="0 -0.11315 0" rpy="${0.5*pi} 0 0" />
-    <axis xyz="0 0 1" />
-<!--limit-->
-    <limit lower="${-1.5*pi}" upper="${1.5*pi}" velocity="3.92" effort="80" />
-  </joint>
-  <link name="${prefix}link_6">
-    <visual>
-      <geometry>
-        <mesh filename="package://tmr_description/meshes/tm5-900/visual/tmr_ee.${format}" />
-      </geometry>
-      <material name="${color}" />
-    </visual>
-    <collision>
-      <geometry>
-        <mesh filename="package://tmr_description/meshes/tm5-900/collision/tmr_ee_c.stl" />
-      </geometry>
-    </collision>
-<!--inertial-->
-    <xacro:cylinder_inertial_z radius="0.045" length="0.06" mass="${mass_6}">
-      <origin xyz="0 0 0" rpy="0 0 0" />
-    </xacro:cylinder_inertial_z>
-  </link>
-  <link name="${prefix}base" />
-  <joint name="${prefix}base_fixed_joint" type="fixed">
-    <parent link="${prefix}base" />
-    <child link="${prefix}link_0" />
-    <origin xyz="0 0 0" rpy="0 0 0" />
-  </joint>
-  <link name="${prefix}flange" />
-  <joint name="${prefix}flange_fixed_joint" type="fixed">
-    <parent link="${prefix}link_6" />
-    <child link="${prefix}flange" />
-    <origin xyz="0 0 0" rpy="0 0 0" />
-  </joint>
-<!--LinkDescription-->
-  </xacro:macro>
-</robot>
+/home/gy/Omron_TM_ROS2/tmr_description/xacro/macro.tm5-900.urdf.xacro

File: install/tmr_description/share/tmr_description/xacro/macro.transmission.xacro (robot description, xacro)
@@ -1,59 +1 @@
-<?xml version="1.0"?>
-<robot xmlns:xacro="http://wiki.ros.org/xacro">
-  <xacro:macro name="tmr_transmission" params="prefix hw_iface">
-    <transmission name="${prefix}trans_1">
-      <type>transmission_interface/SimpleTransmission</type>
-      <joint name="${prefix}joint_1">
-        <hardwareInterface>${hw_iface}</hardwareInterface>
-      </joint>
-      <actuator name="${prefix}motor_1">
-        <mechanicalReduction>1</mechanicalReduction>
-      </actuator>
-    </transmission>
-    <transmission name="${prefix}trans_2">
-      <type>transmission_interface/SimpleTransmission</type>
-      <joint name="${prefix}joint_2">
-        <hardwareInterface>${hw_iface}</hardwareInterface>
-      </joint>
-      <actuator name="${prefix}motor_2">
-        <mechanicalReduction>1</mechanicalReduction>
-      </actuator>
-    </transmission>
-    <transmission name="${prefix}trans_3">
-      <type>transmission_interface/SimpleTransmission</type>
-      <joint name="${prefix}joint_3">
-        <hardwareInterface>${hw_iface}</hardwareInterface>
-      </joint>
-      <actuator name="${prefix}motor_3">
-        <mechanicalReduction>1</mechanicalReduction>
-      </actuator>
-    </transmission>
-    <transmission name="${prefix}trans_4">
-      <type>transmission_interface/SimpleTransmission</type>
-      <joint name="${prefix}joint_4">
-        <hardwareInterface>${hw_iface}</hardwareInterface>
-      </joint>
-      <actuator name="${prefix}motor_4">
-        <mechanicalReduction>1</mechanicalReduction>
-      </actuator>
-    </transmission>
-    <transmission name="${prefix}trans_5">
-      <type>transmission_interface/SimpleTransmission</type>
-      <joint name="${prefix}joint_5">
-        <hardwareInterface>${hw_iface}</hardwareInterface>
-      </joint>
-      <actuator name="${prefix}motor_5">
-        <mechanicalReduction>1</mechanicalReduction>
-      </actuator>
-    </transmission>
-    <transmission name="${prefix}trans_6">
-      <type>transmission_interface/SimpleTransmission</type>
-      <joint name="${prefix}joint_6">
-        <hardwareInterface>${hw_iface}</hardwareInterface>
-      </joint>
-      <actuator name="${prefix}motor_6">
-        <mechanicalReduction>1</mechanicalReduction>
-      </actuator>
-    </transmission>
-  </xacro:macro>
-</robot>
+/home/gy/Omron_TM_ROS2/tmr_description/xacro/macro.transmission.xacro

File: install/tmr_description/share/tmr_description/xacro/tm5-900.urdf.xacro (robot description, xacro)
@@ -1,40 +1 @@
-<?xml version="1.0"?>
-<robot xmlns:xacro="http://wiki.ros.org/xacro" name="tm5-900">
-  <xacro:arg name="ns" default="" />
-  <xacro:arg name="prefix" default="" />
-  <xacro:arg name="gripper" default="none" />
-  <xacro:arg name="color" default="none" />
-  <xacro:arg name="trans_hw_iface" default="hardware_interface/PositionJointInterface" />
-  <xacro:include filename="$(find tmr_description)/xacro/macro.gazebo.xacro" />
-  <xacro:include filename="$(find tmr_description)/xacro/macro.transmission.xacro" />
-  <xacro:include filename="$(find tmr_description)/xacro/macro.materials.xacro" />
-  <!-- tm5-900 -->
-  <xacro:include filename="$(find tmr_description)/xacro/macro.tm5-900.urdf.xacro" />
-  <!--  -->
-  <xacro:tmr_gazebo ns="$(arg ns)" prefix="$(arg prefix)" />
-  <xacro:tmr_transmission prefix="$(arg prefix)" hw_iface="$(arg trans_hw_iface)" />
-  <xacro:tmr_materials/>
-  <!-- Arm -->
-  <xacro:property name="color" value="$(arg color)"/>
-  <xacro:if value="${color == 'none'}">
-    <xacro:tm5-900 ns="$(arg ns)" prefix="$(arg prefix)" />
-  </xacro:if>
-  <!-- Arm.color.stl -->
-  <xacro:unless value="${color == 'none'}">
-    <xacro:tm5-900 ns="$(arg ns)" prefix="$(arg prefix)" color="${color}" format="stl" />
-  </xacro:unless>
-  <!-- Arm + Gripper -->
-  <xacro:property name="gripper" value="$(arg gripper)"/>
-  <xacro:if value="${gripper == 'robotiq_2f'}">
-    <xacro:include filename="$(find tmr_description)/xacro/gripper/robotiq_2f.urdf.xacro" />
-    <xacro:robotiq_2f prefix="$(arg prefix)"/>
-  </xacro:if>
-<!--
-  <link name="world"/>
-  <joint name="world_joint" type="fixed">
-    <parent link="world" />
-    <child link="$(arg prefix)base"/>
-    <origin xyz="0 0 0" rpy="0 0 0"/>
-  </joint>
--->
-</robot>
+/home/gy/Omron_TM_ROS2/tmr_description/xacro/tm5-900.urdf.xacro
