Commit message: fix pathing issue, add destination publisher, add rviz config

File: src/tm_models/urdf/tm12.urdf (robot description, URDF)
Before this commit: robot tm12, 11 links, 10 joints
Links:
- added link EOAT; collision mesh filename=package://tmr_description/meshes/gripper/robotiq/2f-85/robo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; visual mesh filename=package://tmr_description/meshes/gripper/robotiq/2f-85/robo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
Joints:
- added joint joint_EOAT: type fixed, parent flange_link, child EOAT, origin xyz=0 0 0 rpy=0 0 0, axis 0 0 0
